File: Hardware/ESP32-Based/CONTROLLER_BOARD/ROBOTIC_ARM.kicad_pcb (KiCad board)
At the start: 2 copper layers, 55.7 x 50 mm, 29 parts, among them J1 Screw_Terminal_01x02, J10 USB_C_Receptacle_USB2.0_16P, J2 Conn_01x03_Pin, J3 Conn_01x03_Pin, J4 Conn_01x03_Pin, J5 Conn_01x03_Pin, J6 Conn_01x03_Pin, J7 Conn_01x03_Pin, J8 Conn_01x03_Pin, J9 Conn_01x03_Pin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

Commit message: Update on PCB design
Routing:
- added copper zone on B.Cu, net GND
- added copper zone on F.Cu, net GND
Other:
- board size 55.7 x 50 mm -> 55.7 x 43.7 mm
Changed lines of the file:
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@@
 	)
 	(gr_rect
-		(start 133 72.48)
+		(start 133 78.81)
 		(end 188.7 122.5)
 		(stroke
@@
 		(net 65)
 	)
+	(zone
+		(net 1)
+		(net_name "GND")
+		(layer "F.Cu")
+		(hatch edge 0.5)
+		(priority 1)
+		(connect_pads
+			(clearance 0.5)
+		)
+		(min_thickness 0.25)
+		(filled_areas_thickness no)
+		(fill yes
+			(thermal_gap 0.5)
+			(thermal_bridge_width 0.5)
+		)
+		(polygon
+			(pts
+				(xy 133 78.81) (xy 188.7 78.81) (xy 188.7 122.5) (xy 133 122.5)
+			)
+		)
+	)
+	(zone
+		(net 1)
+		(net_name "GND")
+		(layer "B.Cu")
+		(hatch edge 0.5)
+		(connect_pads
+			(clearance 0.5)
+		)
+		(min_thickness 0.25)
+		(filled_areas_thickness no)
+		(fill yes
+			(thermal_gap 0.5)
+			(thermal_bridge_width 0.5)
+		)
+		(polygon
+			(pts
+				(xy 133.01 78.82) (xy 133 122.49) (xy 188.7 122.5) (xy 188.7 78.81)
+			)
+		)
+	)
 	(embedded_fonts no)
